Commit message: add middle plating to gate urdf file

File: sim/urdf/gate.urdf (robot description, URDF)
Before this commit: robot gate, 3 links, 2 joints
Links:
- added link middle_plating
Joints:
- added joint back_middle_joint: type fixed, parent back_plating, child middle_plating

Commit message: add generic dimensions

File: sim/urdf/gate.urdf (robot description, URDF)
Before this commit: robot gate, 4 links, 3 joints
Links:
- removed link back_plating
- added link top_plating
Joints:
- removed joint back_left_joint
- removed joint back_middle_joint
- removed joint back_right_joint
- added joint top_left_joint: type fixed, parent top_plating, child left_plating, origin xyz=0 0 0
- added joint top_middle_joint: type fixed, parent top_plating, child middle_plating, origin xyz=10 0 0
- added joint top_right_joint: type fixed, parent top_plating, child right_plating, origin xyz=4 0 0
